Commit message: URDF Update
Added two support plates so they are visible in rviz

File: urdf/macros/sample_description.xacro (robot description, xacro)
@@ -151,4 +151,40 @@
         xyz="0 0 0" />
     </joint>
+    <link name="${prefix}_support_one">
+      <visual>
+        <geometry>
+          <box size="1.5 0.3 0.01"/>
+        </geometry>
+        <origin rpy="0 0 0" xyz="-0.75 0.15 -0.005"/>
+        <material
+          name="">
+          <color
+            rgba="0.2 0.2 0.2 1" />
+        </material>
+      </visual>
+    </link>
+    <joint name="${prefix}_to_support_one" type="fixed">
+      <parent link="${prefix}_link"/>
+      <child link="${prefix}_support_one"/>
+      <origin rpy="0 0 3.14159" xyz="-0.05 -0.35 0"/>
+    </joint>
+    <link name="${prefix}_support_two">
+      <visual>
+        <geometry>
+          <box size="1.5 0.3 0.01"/>
+        </geometry>
+        <origin rpy="0 0 0" xyz="-0.75 0.15 -0.005"/>
+        <material
+          name="">
+          <color
+            rgba="0.2 0.2 0.2 1" />
+        </material>
+      </visual>
+    </link>
+    <joint name="${prefix}_to_support_two" type="fixed">
+      <parent link="${prefix}_link"/>
+      <child link="${prefix}_support_two"/>
+      <origin rpy="0 0 3.14159" xyz="-0.05 -0.65 0"/>
+    </joint>
   </xacro:macro>
 </robot>
